File: AttinyXXX6-Minimal-DEV-BOARD.kicad_sch (KiCad schematic)
At the start: 15 parts, among them J1 USB_B_Micro, J2 PWR_CONN, J3 UPDI, J4 Conn, J5 Conn, SW1 SW, U1 ATtinyXXX6

Commit message: pinout and updi
PIN B0 location change and UPDI connector pin change to universal one.
Connections:
- net A0: now also J3.1 (Pin_1); no longer J3.6 (Pin_6)
- net B0: now also J5.5 (Pin_5); no longer J4.9 (Pin_9)
- net B1: now also J5.6 (Pin_6); no longer J5.5 (Pin_5)
- net B2: now also J3.5 (Pin_5), J5.7 (Pin_7); no longer J3.2 (Pin_2), J5.6 (Pin_6)
- net B3: now also J5.8 (Pin_8); no longer J5.7 (Pin_7)
- net B4: now also J5.9 (Pin_9); no longer J5.8 (Pin_8)
- net B5: now also J4.9 (Pin_9); no longer J5.9 (Pin_9)
- net GND: now also J3.6 (Pin_6); no longer J3.3 (Pin_3), J3.5 (Pin_5)
- net VCC: now also J3.2 (Pin_2); no longer J3.1 (Pin_1)
- no-connect marks 3 -> 4
Changed lines of the file:
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@@
 (kicad_sch (version 20211123) (generator eeschema)
   (paper "A4")
+  (title_block
+    (date "2022-10-10")
+    (rev "0.0.2")
+  )
   (junction (at 66.04 57.15) (diameter 0) (color 0 0 0 0)
   )
@@
   (no_connect (at 74.93 46.99))
   (no_connect (at 74.93 44.45))
+  (no_connect (at 120.65 81.28))
   (wire (pts (xy 241.3 110.49) (xy 246.38 110.49))
     (stroke (width 0) (type default) (color 0 0 0 0))
@@
     (stroke (width 0) (type default) (color 0 0 0 0))
   )
-  (wire (pts (xy 116.84 81.28) (xy 120.65 81.28))
-    (stroke (width 0) (type default) (color 0 0 0 0))
-  )
   (wire (pts (xy 90.17 127) (xy 97.79 127))
     (stroke (width 0) (type default) (color 0 0 0 0))
@@
     (stroke (width 0) (type default) (color 0 0 0 0))
   )
-  (label "A0" (at 137.16 83.82 180)
+  (label "GND" (at 137.16 83.82 180)
     (effects (font (size 1.27 1.27)) (justify right bottom))
   )
@@
     (effects (font (size 1.27 1.27)) (justify right bottom))
   )
-  (label "B0" (at 226.06 120.65 180)
-    (effects (font (size 1.27 1.27)) (justify right bottom))
-  )
-  (label "B2" (at 137.16 78.74 180)
-    (effects (font (size 1.27 1.27)) (justify right bottom))
-  )
-  (label "VCC" (at 116.84 78.74 0)
+  (label "B5" (at 226.06 120.65 180)
+    (effects (font (size 1.27 1.27)) (justify right bottom))
+  )
+  (label "VCC" (at 137.16 78.74 180)
+    (effects (font (size 1.27 1.27)) (justify right bottom))
+  )
+  (label "A0" (at 116.84 78.74 0)
     (effects (font (size 1.27 1.27)) (justify left bottom))
   )
@@
     (effects (font (size 1.27 1.27)) (justify right bottom))
   )
-  (label "B5" (at 241.3 120.65 0)
+  (label "B4" (at 241.3 120.65 0)
     (effects (font (size 1.27 1.27)) (justify left bottom))
   )
@@
     (effects (font (size 1.27 1.27)) (justify right bottom))
   )
-  (label "GND" (at 116.84 83.82 0)
+  (label "B2" (at 116.84 83.82 0)
     (effects (font (size 1.27 1.27)) (justify left bottom))
   )
@@
     (effects (font (size 1.27 1.27)) (justify right bottom))
   )
-  (label "GND" (at 116.84 81.28 0)
-    (effects (font (size 1.27 1.27)) (justify left bottom))
-  )
   (label "B1" (at 97.79 149.86 180)
     (effects (font (size 1.27 1.27)) (justify right bottom))
@@
     (effects (font (size 1.27 1.27)) (justify left bottom))
   )
-  (label "B1" (at 241.3 110.49 0)
+  (label "B0" (at 241.3 110.49 0)
     (effects (font (size 1.27 1.27)) (justify left bottom))
   )
@@
     (effects (font (size 1.27 1.27)) (justify right bottom))
   )
-  (label "B4" (at 241.3 118.11 0)
+  (label "B3" (at 241.3 118.11 0)
     (effects (font (size 1.27 1.27)) (justify left bottom))
   )
@@
     (effects (font (size 1.27 1.27)) (justify left bottom))
   )
-  (label "B2" (at 241.3 113.03 0)
+  (label "B1" (at 241.3 113.03 0)
     (effects (font (size 1.27 1.27)) (justify left bottom))
   )
@@
     (effects (font (size 1.27 1.27)) (justify left bottom))
   )
-  (label "B3" (at 241.3 115.57 0)
-    (effects (font (size 1.27 1.27)) (justify left bottom))
-  )
+  (label "B2" (at 241.3 115.57 0)
+    (effects (font (size 1.27 1.27)) (justify left bottom))
+  )
